File: Pico_LoRa.kicad_pcb (KiCad board)
At the start: 4 copper layers, 56.6 x 57.7 mm, 46 parts, among them IC1 MCP73871, IC2 XB8089D, IC3 TPS25940x, J1 Conn, J2 Conn, U1 Pico, U2 BMP280, U3 RFM95W-868S2, U4 DS18B20

Commit message: some more GND vias
Routing:
- net GND: vias 36 -> 62
Changed lines of the file:
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@@
     (pad "43" smd rect locked (at 2.54 23.9) (size 3.5 1.7) (drill (offset -0.9 0)) (layers "F.Cu" "F.Mask")
       (net 56 "unconnected-(U1-Pad43)") (pinfunction "SWDIO") (pintype "bidirectional+no_connect"))
-    (model "${KICAD6_USER_3DMODELS_DIR}/RP2040--3DModel-STEP-175466.STEP"
-      (offset (xyz 0 0 0))
-      (scale (xyz 1 1 1))
-      (rotate (xyz 0 0 0))
+    (model "${KICAD6_USER_3DMODEL_DIR}/SC0915--3DModel-STEP-56544.STEP"
+      (offset (xyz 0 0 0))
+      (scale (xyz 1 1 1))
+      (rotate (xyz 90 -180 -180))
     )
     (model "${KICAD6_USER_3DMODELS_DIR}/SC0915--3DModel-STEP-56544.STEP"
@@
       (rotate (xyz 0 0 0))
     )
-    (model "${KICAD6_USER_3DMODELS_DIR}/RFM95W-868S2--3DModel-STEP-56544.STEP"
+    (model "${KICAD6_USER_3DMODEL_DIR}/RFM95W-868S2--3DModel-STEP-56544.STEP"
       (offset (xyz 0 0 0))
       (scale (xyz 1 1 1))
@@
   (via (at 94.05 123.95) (size 0.8) (drill 0.4) (layers "F.Cu" "B.Cu") (free) (net 5))
   (via (at 83.625 82.875) (size 0.8) (drill 0.4) (layers "F.Cu" "B.Cu") (net 5))
+  (via (at 128.1 83) (size 0.8) (drill 0.4) (layers "F.Cu" "B.Cu") (free) (net 5))
+  (via (at 113.35 129.25) (size 0.8) (drill 0.4) (layers "F.Cu" "B.Cu") (free) (net 5))
   (via (at 119.425 108.075) (size 0.8) (drill 0.4) (layers "F.Cu" "B.Cu") (free) (net 5))
   (via (at 87.125 100.9) (size 0.8) (drill 0.4) (layers "F.Cu" "B.Cu") (net 5))
@@
   (via (at 106.7 116.975) (size 0.8) (drill 0.4) (layers "F.Cu" "B.Cu") (net 5))
   (via (at 82.4 96.625) (size 0.8) (drill 0.4) (layers "F.Cu" "B.Cu") (net 5))
+  (via (at 100.35 118.5) (size 0.8) (drill 0.4) (layers "F.Cu" "B.Cu") (free) (net 5))
   (via (at 93.625 82.85) (size 0.8) (drill 0.4) (layers "F.Cu" "B.Cu") (net 5))
+  (via (at 100.35 129.25) (size 0.8) (drill 0.4) (layers "F.Cu" "B.Cu") (free) (net 5))
+  (via (at 124.85 118.5) (size 0.8) (drill 0.4) (layers "F.Cu" "B.Cu") (free) (net 5))
   (via (at 128.025 121.975) (size 0.8) (drill 0.4) (layers "F.Cu" "B.Cu") (free) (net 5))
   (via (at 100.375 91.125) (size 0.8) (drill 0.4) (layers "F.Cu" "B.Cu") (free) (net 5))
+  (via (at 100.35 103.5) (size 0.8) (drill 0.4) (layers "F.Cu" "B.Cu") (free) (net 5))
   (via (at 127.975 130.65) (size 0.8) (drill 0.4) (layers "F.Cu" "B.Cu") (free) (net 5))
+  (via (at 87.1 103) (size 0.8) (drill 0.4) (layers "F.Cu" "B.Cu") (free) (net 5))
   (via (at 127.7 94.35) (size 0.8) (drill 0.4) (layers "F.Cu" "B.Cu") (net 5))
   (via (at 100.35 99.3) (size 0.8) (drill 0.4) (layers "F.Cu" "B.Cu") (free) (net 5))
+  (via (at 105.6 95.5) (size 0.8) (drill 0.4) (layers "F.Cu" "B.Cu") (free) (net 5))
+  (via (at 76.35 118.5) (size 0.8) (drill 0.4) (layers "F.Cu" "B.Cu") (free) (net 5))
   (via (at 94 117) (size 0.8) (drill 0.4) (layers "F.Cu" "B.Cu") (net 5))
+  (via (at 84.35 103) (size 0.8) (drill 0.4) (layers "F.Cu" "B.Cu") (free) (net 5))
+  (via (at 113.35 118.5) (size 0.8) (drill 0.4) (layers "F.Cu" "B.Cu") (free) (net 5))
   (via (at 122.225 98.8) (size 0.8) (drill 0.4) (layers "F.Cu" "B.Cu") (net 5))
   (via (at 116.825 89.625) (size 0.8) (drill 0.4) (layers "F.Cu" "B.Cu") (net 5))
@@
   (via (at 79.175 98.15) (size 0.8) (drill 0.4) (layers "F.Cu" "B.Cu") (net 5))
   (via (at 115.525 107.55) (size 0.8) (drill 0.4) (layers "F.Cu" "B.Cu") (free) (net 5))
+  (via (at 123.1 83) (size 0.8) (drill 0.4) (layers "F.Cu" "B.Cu") (free) (net 5))
   (via (at 106.75 124.025) (size 0.8) (drill 0.4) (layers "F.Cu" "B.Cu") (free) (net 5))
   (via (at 78.775 124.025) (size 0.8) (drill 0.4) (layers "F.Cu" "B.Cu") (net 5))
   (via (at 121.925 87.875) (size 0.8) (drill 0.4) (layers "F.Cu" "B.Cu") (net 5))
+  (via (at 113.35 124) (size 0.8) (drill 0.4) (layers "F.Cu" "B.Cu") (free) (net 5))
   (via (at 100.35 95.375) (size 0.8) (drill 0.4) (layers "F.Cu" "B.Cu") (free) (net 5))
   (via (at 124.45 106.5) (size 0.8) (drill 0.4) (layers "F.Cu" "B.Cu") (free) (net 5))
@@
   (via (at 94.025 130.875) (size 0.8) (drill 0.4) (layers "F.Cu" "B.Cu") (net 5))
   (via (at 85.35 87.8) (size 0.8) (drill 0.4) (layers "F.Cu" "B.Cu") (net 5))
+  (via (at 85.6 84.5) (size 0.8) (drill 0.4) (layers "F.Cu" "B.Cu") (free) (net 5))
+  (via (at 78.85 95.5) (size 0.8) (drill 0.4) (layers "F.Cu" "B.Cu") (free) (net 5))
+  (via (at 87.85 129.25) (size 0.8) (drill 0.4) (layers "F.Cu" "B.Cu") (free) (net 5))
+  (via (at 95.35 84.5) (size 0.8) (drill 0.4) (layers "F.Cu" "B.Cu") (free) (net 5))
+  (via (at 81.1 103) (size 0.8) (drill 0.4) (layers "F.Cu" "B.Cu") (free) (net 5))
   (via (at 106.75 130.875) (size 0.8) (drill 0.4) (layers "F.Cu" "B.Cu") (net 5))
+  (via (at 112.6 100.25) (size 0.8) (drill 0.4) (layers "F.Cu" "B.Cu") (free) (net 5))
   (via (at 122.275 101) (size 0.8) (drill 0.4) (layers "F.Cu" "B.Cu") (free) (net 5))
+  (via (at 110.6 89) (size 0.8) (drill 0.4) (layers "F.Cu" "B.Cu") (free) (net 5))
+  (via (at 76.35 129.75) (size 0.8) (drill 0.4) (layers "F.Cu" "B.Cu") (free) (net 5))
+  (via (at 87.85 118.5) (size 0.8) (drill 0.4) (layers "F.Cu" "B.Cu") (free) (net 5))
   (via (at 127.975 113.35) (size 0.8) (drill 0.4) (layers "F.Cu" "B.Cu") (free) (net 5))
+  (via (at 100.35 124) (size 0.8) (drill 0.4) (layers "F.Cu" "B.Cu") (free) (net 5))
+  (via (at 95.35 91) (size 0.8) (drill 0.4) (layers "F.Cu" "B.Cu") (free) (net 5))
+  (via (at 87.85 124) (size 0.8) (drill 0.4) (layers "F.Cu" "B.Cu") (free) (net 5))
   (via (at 89.7 82.85) (size 0.8) (drill 0.4) (layers "F.Cu" "B.Cu") (net 5))
   (via (at 81.325 130.9) (size 0.8) (drill 0.4) (layers "F.Cu" "B.Cu") (net 5))
   (via (at 82.675 100.85) (size 0.8) (drill 0.4) (layers "F.Cu" "B.Cu") (net 5))
+  (via (at 114.35 91.75) (size 0.8) (drill 0.4) (layers "F.Cu" "B.Cu") (free) (net 5))
   (segment (start 81.32 130.905) (end 81.325 130.9) (width 0.25) (layer "B.Cu") (net 5))
   (segment (start 101.775 88.1) (end 104.075 85.8) (width 0.25) (layer "F.Cu") (net 6))
